File: hardware/athena.kicad_sch (KiCad schematic)
At the start: 3 parts, among them U1 INA226AIDGSR, U2 STM32H755ZIT6

Commit message: v2
Parts:
- added AE1: 2450AT18A100E, lcsc:ANT-SMD_L3.2-W1.6, symbol lcsc:2450AT18A100E
- added C1, C19, C20: 4.7uF, symbol Device:C
- added C10, C11, C13, C15, C16, C5, C6, C8: 100nF, Capacitor_SMD:C_0402_1005Metric, symbol Device:C
- added C12, C7, C9: 4.7uF, Capacitor_SMD:C_0603_1608Metric, symbol Device:C
- added C14, C17: 1uF, Capacitor_SMD:C_0402_1005Metric, symbol Device:C
- added C18, C2, C3, C4: 10pF, Capacitor_SMD:C_0402_1005Metric, symbol Device:C
- added C21, C23: 10uF, symbol Device:C
- added C22: 47nF, symbol Device:C
- added Card1: TF-01A, lcsc:TF-SMD_TF-01A, symbol lcsc:TF-01A
- added D1, D2, D3, D4: 1N4148WS, Diode_SMD:D_SOD-323, symbol Diode:1N4148WS
- added D5: LED, LED_SMD:LED_0402_1005Metric, symbol Device:LED
- added FL1: MLPF-WB55-01E3, lcsc:FILTER-SMD_6P-L1.6-W1.0-P0.50-BL, symbol lcsc:MLPF-WB55-01E3
- added L1: 10uH, Inductor_SMD:L_0603_1608Metric, symbol Device:L
- added L2: 10nH, Inductor_SMD:L_0603_1608Metric, symbol Device:L
- added L3: 1239AS-H-1R0M=P2, lcsc:L1008, symbol lcsc:1239AS-H-1R0M=P2
- added R1, R2: 5.1K, symbol Device:R
- added R10: 5.7K, symbol Device:R
- added R11: 5.23K, symbol Device:R
- added R12: 30.1K, symbol Device:R
- added R13: 10K, symbol Device:R
- added R3, R5: 10K, Resistor_SMD:R_0402_1005Metric, symbol Device:R
- added R4: 150, Resistor_SMD:R_0402_1005Metric, symbol Device:R
- added R6, R7: 2.2K, symbol Device:R
- added R8: 383R, symbol Device:R
- added R9: 150K, symbol Device:R
- added RF1: BWSMA-KWE-Z001, lcsc:SMA-TH_BWSMA-KWE-Z001, symbol lcsc:BWSMA-KWE-Z001
- added SW1, SW2: SW_Push, lcsc:SW-SMD_L3.9-W3.0-P4.45, symbol Switch:SW_Push
- added TP1, TP2, TP3: TestPoint, TestPoint:TestPoint_Pad_1.0x1.0mm, symbol Connector:TestPoint
- added U10: STM32WB55RGVx, Package_DFN_QFN:QFN-68-1EP_8x8mm_P0.4mm_EP6.4x6.4mm, symbol MCU_ST_STM32WB:STM32WB55RGVx
- added U11: SX1262IMLTRT, lcsc:QFN-24_L4.0-W4.0-P0.50-BL-EP2.6, symbol lcsc:SX1262IMLTRT
- added U12: TPS7A2033PDBVR, lcsc:SOT-23-5_L2.9-W1.6-P0.95-LS2.8-BR, symbol lcsc:TPS7A2033PDBVR
- added U13: TPS563209DDCR, lcsc:SOT-23-6_L2.9-W1.6-P0.95-LS2.8-BR, symbol lcsc:TPS563209DDCR
- added U14: TPS630701RNMR, lcsc:VQFN-HR-15_L3.0-W2.5-P0.50-BL_TPS63070RNMR, symbol lcsc:TPS630701RNMR
- added U15: W25Q128JVSIQ, lcsc:SOIC-8_L5.3-W5.3-P1.27-LS8.0-BL, symbol lcsc:W25Q128JVSIQ
- added U16: TPD2EUSB30, Package_TO_SOT_SMD:Texas_DRT-3, symbol Power_Protection:TPD2EUSB30
- added U17: NX2012SA-32.768KHZ-STD-MUB-2, lcsc:CRYSTAL-SMD_L2.0-W1.2, symbol lcsc:NX2012SA-32.768KHZ-STD-MUB-2
- added U18: BQ25886RGE, Package_DFN_QFN:Texas_RGE0024H_VQFN-24-1EP_4x4mm_P0.5mm_EP2.7x2.7mm, symbol Battery_Management:BQ25886RGE
- added U19, U22: SZYY0402Y_C434450, lcsc:LED0402-FD_YELLOW, symbol lcsc:SZYY0402Y_C434450
- added U20: USB2422T-I/MJ, lcsc:QFN-24_L4.0-W4.0-P0.50-TL-EP2.5, symbol lcsc:USB2422T-I_MJ
- added U21, U5: BMP581, lcsc:LGA-10_L2.0-W2.0-P0.50-TL_BMP581, symbol lcsc:BMP581
- added U3: BMI270, lcsc:LGA-14_L3.0-W2.5-P0.50-BR, symbol lcsc:BMI270
- added U4: BMM350_C17225907, lcsc:WLCSP-9_L1.3-W1.3-R3-C3-P0.40-TL, symbol lcsc:BMM350_C17225907
- added U6: H3LIS331DLTR, lcsc:LGA-16_L3.0-W3.0-P0.50-BL, symbol lcsc:H3LIS331DLTR
- added U7: ICM-42688-P, lcsc:LGA-14_L3.0-W2.5-P0.50-TL, symbol lcsc:ICM-42688-P
- added U8: MAX-M10S-00B, lcsc:SMD-18_L10.1-W9.7-P1.10-TL_SKG09F, symbol lcsc:MAX-M10S-00B
- added U9: MIA-M10Q-00B, lcsc:LGA-53_L4.5-W4.5-R9-C9-P0.50-TL_MIA-M10Q, symbol lcsc:MIA-M10Q-00B
- added X1: NX2016SA-32MHZ-STD-CZS-5, lcsc:OSC-SMD_4P-L2.0-W1.6-BL, symbol lcsc:NX2016SA-32MHZ-STD-CZS-5
Connections:
- net GND: now reaches USB1.1 (GND)
- net GND: now also USB1.12 (GND), USB1.13 (SHELL), USB1.14 (SHELL), C1.2, C10.2, C11.2, C12.2, C13.2, C14.2, C15.2, C16.2, C17.2, C18.2, C19.2, C2.2, C20.2, C21.2, C23.2, C3.2, C4.2, C5.2, C6.2, C7.2, C8.2, C9.2, FL1.2 (GND4), FL1.4 (GND1), FL1.5 (GND2), FL1.6 (GND3), R1.2, R10.1, R12.1, R13.1, R2.2, R3.1, R8.1, R9.1, SW2.2, TP3.1, U10.32 (VSSRF), U10.42 (VSSSMPS), U10.69 (VSS), U16.3 (GND), U18.19 (GND), U18.20 (GND), U18.25 (GND), U18.4 (GND), U19.2 (K), X1.2 (GND), X1.4 (GND)
- net at USB1.10 (CC2): now also R1.1
- net VBUS: now reaches USB1.11 (VBUS)
- net VBUS: now also USB1.2 (VBUS), C1.1, C19.1, U18.23 (VBUS)
- net at USB1.4 (CC1): now also R2.1
- net USB_DN: now reaches USB1.5 (DN2)
- net USB_DN: now also USB1.7 (DN1), U16.2 (D-)
- net USB_DP: now reaches USB1.6 (DP1)
- net USB_DP: now also USB1.8 (DP2), U16.1 (D+)
- new net: C7.1, L1.2, U10.41 (VFBSMPS)
- new net: L2.1, U10.43 (VLXSMPS)
- new net: AE1.1 (ANT), FL1.1 (OUT)
- new net: R10.2, U18.10 (ICHGSET)
- new net: C22.2, U18.12 (BTST)
- new net: U18.15 (SYS), U18.16 (SYS)
- new net: C22.1, U18.17 (SW), U18.18 (SW)
- new net: U18.2 (STAT), U22.2 (K)
- new net: U18.21 (PMID), U18.22 (PMID)
- new net: R9.2, U18.6 (VSET)
- new net: R11.1, R12.2, R13.2, U18.7 (TS)
- new net: R8.2, U18.8 (ILIM)
- new net: D5.1 (K), U18.9 (~{PG})
- new net: R4.1, U19.1 (A)
- new net: D1.1 (K), D2.1 (K), R5.2, SW2.1
- new net: R7.1, U22.1 (A)
- new net: D5.2 (A), R6.1
- new net: L1.1, L2.2
- new net: D3.1 (K), D4.1 (K), R3.2, SW1.1
- new net +3.3V: C10.1, C11.1, C12.1, C13.1, C14.1, C15.1, C16.1, C17.1, C5.1, C6.1, C8.1, C9.1, R5.1, SW1.2, U10.1 (VBAT), U10.13 (VREF+), U10.14 (VDDA), U10.30 (VDD), U10.33 (VDDRF), U10.44 (VDDSMPS), U10.45 (VDD), U10.55 (VDDUSB), U10.68 (VDD)
- new net +BATT: C21.1, U18.13 (BAT), U18.14 (BAT)
- new net BOOT_MPU: D3.2 (A)
- new net BOOT_TPU: D4.2 (A), U10.5 (PH3)
- new net BQ_VREGN: C20.1, R11.2, R6.2, R7.2, U18.11 (REGN)
- new net HXIN: U10.35 (OSC_IN)
- new net HXOUT: U10.34 (OSC_OUT)
- new net LXIN: U10.3 (PC14)
- new net LXOUT: U10.4 (PC15)
- new net RESET_MPU: D2.2 (A)
- new net RESET_TPU: D1.2 (A), U10.8 (NRST)
- new net RF: FL1.3 (IN), U10.31 (RF1)
- new net TPU_DN: U10.52 (PA11)
- new net TPU_DP: U10.53 (PA12)
- new net TPU_HXIN: C2.1, X1.1
- new net TPU_HXOUT: C3.1, X1.3
- new net TPU_LED: R4.2, U10.2 (PC13)
- new net TPU_LXIN: C4.1, U17.1 (OSC1)
- new net TPU_LXOUT: C18.1, U17.2 (OSC2)
- new net TPU_SWCLK: TP2.1, U10.56 (PA14)
- new net TPU_SWDIO: TP1.1, U10.54 (PA13)
- no-connect marks 0 -> 7
Other:
- moved on the sheet: U1, U2, USB1

Commit message: aaaaa
Parts:
- removed U2: STM32H755ZIT6, lcsc:LQFP-144_L20.0-W20.0-P0.50-LS22.0-BL, symbol lcsc:STM32H755ZIT6
- added U23: STM32H755ZITx, Package_QFP:LQFP-144_20x20mm_P0.5mm, symbol MCU_ST_STM32H7:STM32H755ZITx
Connections:
- net +3.3V: now also C20.1, U18.11 (REGN)
- net BQ_VREGN: no longer C20.1, U18.11 (REGN)
- net at L3.1: now also C23.1, U18.21 (PMID), U18.22 (PMID)
- net at L3.2: now also C22.1, U18.17 (SW), U18.18 (SW)
- new net: U23.104 (VSS), U23.118 (VSS), U23.12 (VSS), U23.128 (VSS), U23.141 (VSS), U23.18 (VSS), U23.33 (VSS), U23.41 (VSS), U23.55 (VSS), U23.6 (VSS), U23.69 (VSS), U23.80 (VSS), U23.89 (VSS)
Other:
- moved on the sheet: C19, C20, C21, C22, C23, D5, L3, R10, R11, R12, R13, R6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

Commit message: half of schematic
Parts:
- removed U1: INA226AIDGSR, lcsc:MSOP-10_L3.0-W3.0-P0.50-LS5.0-BL, symbol lcsc:INA226AIDGSR
- removed U14: TPS630701RNMR, lcsc:VQFN-HR-15_L3.0-W2.5-P0.50-BL_TPS63070RNMR, symbol lcsc:TPS630701RNMR
- removed U15: W25Q128JVSIQ, lcsc:SOIC-8_L5.3-W5.3-P1.27-LS8.0-BL, symbol lcsc:W25Q128JVSIQ
- removed U19: SZYY0402Y_C434450, lcsc:LED0402-FD_YELLOW, symbol lcsc:SZYY0402Y_C434450
- removed U23: STM32H755ZITx, Package_QFP:LQFP-144_20x20mm_P0.5mm, symbol MCU_ST_STM32H7:STM32H755ZITx
- removed U9: MIA-M10Q-00B, lcsc:LGA-53_L4.5-W4.5-R9-C9-P0.50-TL_MIA-M10Q, symbol lcsc:MIA-M10Q-00B
- added C24, C25, C63, C64: 10uF, Capacitor_SMD:C_0603_1608Metric, symbol Device:C
- added C26: 44uF, Capacitor_SMD:C_0805_2012Metric, symbol Device:C
- added C27, C43, C44, C45, C47, C48, C50, C51, C52, C53, C54, C55, C56, C57, C58, C59, C60, C61, C62, C66, C67, C68, C69, C70, C71, C72, C73, C75: 100nF, Capacitor_SMD:C_0402_1005Metric, symbol Device:C
- added C28, C29: 22uF, Capacitor_SMD:C_0603_1608Metric, symbol Device:C
- added C30, C40: 10pF, Capacitor_SMD:C_0402_1005Metric, symbol Device:C
- added C31, C32, C33, C35: 1uF, Capacitor_SMD:C_0402_1005Metric_Pad0.74x0.62mm_HandSolder, symbol Device:C
- added C34: 100nF, Capacitor_SMD:C_0402_1005Metric_Pad0.74x0.62mm_HandSolder, symbol Device:C
- added C36, C37, C38, C39: 15pF C0G, Capacitor_SMD:C_0402_1005Metric_Pad0.74x0.62mm_HandSolder, symbol Device:C
- added C41, C42, C65, C76: 2.2uF, Capacitor_SMD:C_0402_1005Metric, symbol Device:C
- added C46: 1uF, Capacitor_SMD:C_0402_1005Metric, symbol Device:C
- added C49: 4.7uF, Capacitor_SMD:C_0603_1608Metric, symbol Device:C
- added C74: 10nF, Capacitor_SMD:C_0402_1005Metric, symbol Device:C
- added L5: FNR4030S3R3MT, lcsc:IND-SMD_L4.0-W4.0_FNR40XXS, symbol lcsc:FNR4030S3R3MT
- added L6, L7: BLM15AX601SN1D, lcsc:L0402, symbol lcsc:BLM15AX601SN1D
- added R14, R16, R29, R30, R31, R32, R33, R34, R35, R36, R37: 10K, Resistor_SMD:R_0402_1005Metric, symbol Device:R
- added R15: 33.2K, Resistor_SMD:R_0402_1005Metric, symbol Device:R
- added R17, R18, R19: 50K, Resistor_SMD:R_0402_1005Metric, symbol Device:R
- added R20: 12K, Resistor_SMD:R_0402_1005Metric, symbol Device:R
- added R21, R22: 100K, Resistor_SMD:R_0402_1005Metric, symbol Device:R
- added R23, R24, R25, R26, R27, R28: 100R, Resistor_SMD:R_0402_1005Metric, symbol Device:R
- added R39, R40: 4.7K, Resistor_SMD:R_0402_1005Metric, symbol Device:R
- added U1, U14: XL-1608RGBC, lcsc:LED-SMD_4P-L1.6-W0.8-BL, symbol lcsc:XL-1608RGBC
- added U19: NX2012SA-32.768KHZ-STD-MUB-2, lcsc:CRYSTAL-SMD_L2.0-W1.2, symbol lcsc:NX2012SA-32.768KHZ-STD-MUB-2
- added U2: STM32F405VGTx, Package_QFP:LQFP-100_14x14mm_P0.5mm, symbol MCU_ST_STM32F4:STM32F405VGTx
- added U9: W25Q128JVP, Package_SON:WSON-8-1EP_6x5mm_P1.27mm_EP3.4x4.3mm, symbol Memory_Flash:W25Q128JVP
- added X2, X3: XL2EL89COI-111YLC-24M, lcsc:CRYSTAL-SMD_4P-L3.2-W2.5-BL, symbol lcsc:XL2EL89COI-111YLC-24M
- C1, C19, C20, C21, C23: footprint (none) -> Capacitor_SMD:C_0603_1608Metric
- C22: footprint (none) -> Capacitor_SMD:C_0402_1005Metric
- R1, R10, R11, R12, R13, R2, R6, R7, R8, R9: footprint (none) -> Resistor_SMD:R_0402_1005Metric
- R4: value 150 -> 10K; LCSC C25082 -> (none)
Connections:
- net HXIN is gone; now on net TPU_HXIN: U10.35 (OSC_IN)
- net HXOUT is gone; now on net TPU_HXOUT: U10.34 (OSC_OUT)
- net LXIN is gone; now on net TPU_LXIN: U10.3 (PC14)
- net LXOUT is gone; now on net TPU_LXOUT: U10.4 (PC15)
- net +3.3V: now also Card1.4 (VDD), U12.1 (IN), U12.3 (EN), U20.1 (VDD33), U20.18 (VDD33), U20.9 (VDD33), C28.1, C29.1, C32.1, C33.1, C34.1, C43.1, C44.1, C45.1, C46.1, C47.1, C48.1, C49.1, C50.1, C51.1, C52.1, C53.1, C54.1, C55.1, C56.1, C57.1, C58.1, C59.1, C60.1, C61.1, C62.1, C63.1, C64.1, L5.2, L6.2, L7.2, R15.2, R19.2, R29.2, R30.2, R31.2, R32.2, R33.2, R34.2, R35.2, R36.2, R37.2, R39.2, R40.2, U1.3 (com), U14.3 (com), U2.100 (VDD), U2.11 (VDD), U2.19 (VDD), U2.21 (VREF+), U2.28 (VDD), U2.50 (VDD), U2.6 (VBAT), U2.75 (VDD), U9.8 (VCC); no longer U10.14 (VDDA)
- net BOOT_MPU: now also U2.94 (BOOT0)
- net GND: now also Card1.10 (GND), Card1.11 (GND), Card1.12 (GND), Card1.13 (GND), Card1.6 (VSS), U12.2 (GND), U13.1 (GND), U3.6 (GNDIO), U3.7 (GND), U4.B1 (GND), U4.B2 (ADSEL), U4.C3 (BYPASS), U5.3 (VSS), U5.8 (VSS), U5.9 (VSS), U6.10 (Reserved), U6.12 (GND), U6.13 (GND), U6.15 (Reserved), U6.16 (GND), U6.5 (GND), U7.6 (GND), C24.2, C25.2, C26.2, C28.2, C29.2, C30.2, C31.2, C32.2, C33.2, C34.2, C35.2, C36.2, C37.2, C38.2, C39.2, C40.2, C41.2, C42.2, C43.2, C44.2, C45.2, C46.2, C47.2, C48.2, C49.2, C50.2, C51.2, C52.2, C53.2, C54.2, C55.2, C56.2, C57.2, C58.2, C59.2, C60.2, C61.2, C62.2, C63.2, C64.2, C65.1, C66.2, C67.2, C68.2, C69.2, C70.1, C71.1, C72.1, C73.2, C74.2, C75.2, C76.2, R16.1, R17.2, R18.2, R20.2, R22.2, U2.10 (VSS), U2.20 (VSSA), U2.27 (VSS), U2.74 (VSS), U2.99 (VSS), U9.4 (GND), U9.9 (EP), X2.2 (GND), X2.4 (GND), X3.2 (GND), X3.4 (GND)
- net RESET_MPU: now also U2.14 (NRST)
- net TPU_DN: now also U20.4 (USBDM_DN2/PRT_DIS_M2)
- net TPU_DP: now also U20.5 (USBDP_DN2/PRT_DIS_P2)
- net USB_DN: now also U20.19 (USBDM_UP)
- net USB_DP: now also U20.20 (USBDP_UP)
- net VBUS: now also R21.2, R22.1
- net IMU_MISO: now reaches U3.1 (SDO)
- net IMU_MISO: now also U7.1 (AP_SDO/AP_AD0), U2.31 (PA6)
- net BMI_CS: now reaches U3.12 (CSB)
- net BMI_CS: now also R4.1
- net IMU_SCK: now reaches U3.13 (SCX)
- net IMU_SCK: now also U7.13 (AP_SCL/AP_SCLK), U2.30 (PA5)
- net IMU_MOSI: now reaches U3.14 (SDX)
- net IMU_MOSI: now also U7.14 (AP_SDA/AP_SDIO/AP_SDI), U2.32 (PA7)
- net BMI_INT1: now reaches U3.4 (INT1)
- net BMI_INT1: now also U2.33 (PC4)
- net +3.3V_LDO: now reaches U3.5 (VDDIO)
- net +3.3V_LDO: now also R4.2, U12.5 (OUT), U3.8 (VDD), U4.B3 (VDDIO), U4.C1 (VDD), U5.1 (VDDIO), U5.10 (VDD), U6.1 (Vdd_IO), U6.14 (Vdd), U7.5 (VDDIO), U7.8 (VDD), C31.1, C66.1, C67.1, C68.1, C69.1, C70.2, C71.2, C72.2, C73.1, C74.1, C75.1, C76.1
- net BMI_INT2: now reaches U3.9 (INT2)
- net BMI_INT2: now also U2.34 (PC5)
- net ICM_CS: now reaches U7.12 (AP_CS)
- net ICM_CS: now also U2.37 (PB2)
- net ICM_INT: now reaches U7.4 (INT1/INT)
- net ICM_INT2: now reaches U7.9 (INT2/FSYNC/CLKIN)
- net ICM_INT2: now also U2.39 (PE8)
- net SYS: now reaches U18.15 (SYS), U18.16 (SYS)
- net SYS: now also U13.3 (VIN), C24.1, C25.1, C26.1, R14.2
- net HLI_INT1: now reaches U6.11 (INT1)
- net HLI_INT1: now also U2.58 (PD11)
- net SENSOR_SCK: now reaches U6.4 (SCL/SPS)
- net SENSOR_SCK: now also U5.2 (SCK), U2.52 (PB13)
- net SENSOR_MOSI: now reaches U6.6 (SDA/SDI/SDO)
- net SENSOR_MOSI: now also U5.4 (SDI), U2.54 (PB15)
- net SENSOR_MISO: now reaches U6.7 (SDO/SA0)
- net SENSOR_MISO: now also U5.5 (SDO), U2.53 (PB14)
- net HLI_CS: now reaches U6.8 (CS)
- net HLI_CS: now also U2.57 (PD10)
- net HLI_INT2: now reaches U6.9 (INT2)
- net HLI_INT2: now also U2.59 (PD12)
- net at Card1.1 (DAT2(RSV)): now also R31.1
- net at Card1.2 (CDDAT3(CS)): now also R32.1
- net SD_CMD: now reaches Card1.3 (CMD(DI))
- net SD_CMD: now also R33.1, U2.83 (PD2)
- net SD_CLK: now reaches Card1.5 (CLK(SCLK))
- net SD_CLK: now also U2.80 (PC12)
- net SD_D0: now reaches Card1.7 (DAT0(D0))
- net SD_D0: now also R29.1, U2.65 (PC8)
- net at Card1.8 (DAT1(RSV)): now also R30.1
- net SD_CD: now reaches Card1.9 (CD)
- net SD_CD: now also R34.1, U2.82 (PD1)
- net at U13.2 (SW): now also C27.1, L5.1
- net at U13.4 (VFB): now also R15.1, R16.2
- net at U13.5 (EN): now also R14.1
- net at U13.6 (VBST): now also C27.2
- net MAG_INT: now reaches U4.A1 (INT)
- net MAG_INT: now also U2.46 (PE15)
- net MAG_SDA: now reaches U4.A2 (SDA)
- net MAG_SDA: now also R40.1, U2.48 (PB11)
- net MAG_SCL: now reaches U4.A3 (SCK)
- net MAG_SCL: now also R39.1, U2.47 (PB10)
- net at U4.C2 (CRST): now also C65.2
- net BMP_CS: now reaches U5.6 (CSB)
- net BMP_CS: now also U2.55 (PD8)
- net BMP_INT: now reaches U5.7 (INT)
- net BMP_INT: now also U2.56 (PD9)
- net at U20.10 (CRFILT): now also C35.1
- net at U20.13 (SMBDATA/NON_REM1): now also R19.1
- net at U20.14 (SMBCLK/CFG_SEL0): now also R18.1
- net at U20.16 (VBUS_DET): now also R21.1
- net at U20.17 (SUSP_IND/LOCAL_PWR/(NON_REM0)): now also R17.1
- net MPU_DN: now reaches U20.2 (USBDM_DN1/PRT_DIS_M1)
- net MPU_DN: now also U2.70 (PA11)
- net USB_XOUT: now reaches U20.21 (XTALOUT/(CLKIN_EN))
- net USB_XOUT: now also C36.1, X2.1
- net USB_XIN: now reaches U20.22 (XTALIN/CLKIN)
- net USB_XIN: now also C37.1, X2.3
- net at U20.24 (RBIAS): now also R20.1
- net MPU_DP: now reaches U20.3 (USBDP_DN1/PRT_DIS_P1)
- net MPU_DP: now also U2.71 (PA12)
- net TPU_LED: no longer names the net of U10.2 (PC13)
- net TPU_LED: no longer R4.2
- new net: R36.1, U9.7 (~{HOLD}/~{RESET}/IO_{3})
- new net: R24.1, U1.4
- new net: R28.1, U14.4
- new net: C42.1, U2.49 (VCAP_1)
- new net: R35.1, U9.3 (~{WP}/IO_{2})
- new net: R26.2, U14.1
- new net: R27.1, U14.2
- new net: R25.2, U1.1
- new net: R23.1, U1.2
- new net: C41.1, U2.73 (VCAP_2)
- new net FLASH_CLK: U9.6 (CLK)
- new net FLASH_CS: R37.1, U2.92 (PB6), U9.1 (~{CS})
- new net FLASH_MISO: U2.90 (PB4), U9.2 (DO/IO_{1})
- new net FLASH_MOSI: U2.91 (PB5), U9.5 (DI/IO_{0})
- new net FLASH_SCK: U2.89 (PB3)
- new net GPS_RX: U2.87 (PD6)
- new net GPS_TX: U2.86 (PD5)
- new net ICM_INT1: U2.38 (PE7)
- new net MOTOR_1: U2.40 (PE9)
- new net MOTOR_2: U2.42 (PE11)
- new net MOTOR_3: U2.44 (PE13)
- new net MOTOR_4: U2.45 (PE14)
- new net MOTOR_5: U2.63 (PC6)
- new net MOTOR_6: U2.64 (PC7)
- new net MOTOR_7: U2.93 (PB7)
- new net MOTOR_8: U2.66 (PC9)
- new net MPU_B: R24.2, U2.25 (PA2)
- new net MPU_G: R23.2, U2.24 (PA1)
- new net MPU_HXIN: C39.1, U2.12 (PH0), X3.3
- new net MPU_HXOUT: C38.1, U2.13 (PH1), X3.1
- new net MPU_LXIN: C30.1, U19.1 (OSC1), U2.8 (PC14)
- new net MPU_LXOUT: C40.1, U19.2 (OSC2), U2.9 (PC15)
- new net MPU_R: R25.1, U2.23 (PA0)
- new net MPU_SWCLK: U2.76 (PA14)
- new net MPU_SWDIO: U2.72 (PA13)
- new net MPU_VDDA: L6.1, U2.22 (VDDA)
- new net TPU_B: R28.2
- new net TPU_G: R27.2
- new net TPU_R: R26.1
- new net TPU_RX: U2.69 (PA10)
- new net TPU_TX: U2.68 (PA9)
- new net TPU_VDDA: L7.1, U10.14 (VDDA)
- no-connect marks 7 -> 26
Other:
- moved on the sheet: C7, D1, D2, D3, D4, L1, R3, R5, RF1, SW1, SW2, U12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
