File: hardware/athena.kicad_sch (KiCad schematic)
At the start: 160 parts, among them SW1 SW_Push, SW2 SW_Push, U1 XL-1608RGBC, U10 STM32WB55RGVx, U11 SX1262IMLTRT, U12 TPS7A2033PDBVR, U13 TPS563209DDCR, U14 XL-1608RGBC, U16 TPD2EUSB30, U17 NX2012SA-32.768KHZ-STD-MUB-2, U18 BQ25886RGE, U19 NX2012SA-32.768KHZ-STD-MUB-2, U2 STM32F405VGTx, U20 USB2422T-I/MJ, U21 BMP581, U22 SZYY0402Y_C434450, U3 BMI270, U4 BMM350_C17225907, U5 BMP581, U6 H3LIS331DLTR, U7 ICM-42688-P, U8 MAX-M10S-00B, U9 W25Q128JVP, X1 NX2016SA-32MHZ-STD-CZS-5, X2 XL2EL89COI-111YLC-24M, X3 XL2EL89COI-111YLC-24M

Commit message: more stuffx
Parts:
- removed AE1: 2450AT18A100E, lcsc:ANT-SMD_L3.2-W1.6, symbol lcsc:2450AT18A100E
- removed C10, C11, C13, C15, C16, C43, C44, C45, C47, C48, C5, C50, C51, C52, C53, C54, C55, C56, C57, C58, C59, C6, C60, C61, C62, C66, C67, C68, C69, C70, C71, C72, C73, C75, C8: 100nF, Capacitor_SMD:C_0402_1005Metric, symbol Device:C
- removed C12, C49, C7, C9: 4.7uF, Capacitor_SMD:C_0603_1608Metric, symbol Device:C
- removed C14, C17, C46: 1uF, Capacitor_SMD:C_0402_1005Metric, symbol Device:C
- removed C18, C2, C3, C30, C4, C40: 10pF, Capacitor_SMD:C_0402_1005Metric, symbol Device:C
- removed C38, C39: 15pF C0G, Capacitor_SMD:C_0402_1005Metric_Pad0.74x0.62mm_HandSolder, symbol Device:C
- removed C41, C42, C65, C76: 2.2uF, Capacitor_SMD:C_0402_1005Metric, symbol Device:C
- removed C63, C64: 10uF, Capacitor_SMD:C_0603_1608Metric, symbol Device:C
- removed C74: 10nF, Capacitor_SMD:C_0402_1005Metric, symbol Device:C
- removed Card1: TF-01A, lcsc:TF-SMD_TF-01A, symbol lcsc:TF-01A
- removed FL1: MLPF-WB55-01E3, lcsc:FILTER-SMD_6P-L1.6-W1.0-P0.50-BL, symbol lcsc:MLPF-WB55-01E3
- removed L1: 10uH, Inductor_SMD:L_0603_1608Metric, symbol Device:L
- removed L2: 10nH, Inductor_SMD:L_0603_1608Metric, symbol Device:L
- removed L6, L7: BLM15AX601SN1D, lcsc:L0402, symbol lcsc:BLM15AX601SN1D
- removed R29, R30, R31, R32, R33, R34, R35, R36, R37, R4: 10K, Resistor_SMD:R_0402_1005Metric, symbol Device:R
- removed R39, R40: 4.7K, Resistor_SMD:R_0402_1005Metric, symbol Device:R
- removed RF1: BWSMA-KWE-Z001, lcsc:SMA-TH_BWSMA-KWE-Z001, symbol lcsc:BWSMA-KWE-Z001
- removed TP1, TP2, TP3: TestPoint, TestPoint:TestPoint_Pad_1.0x1.0mm, symbol Connector:TestPoint
- removed U10: STM32WB55RGVx, Package_DFN_QFN:QFN-68-1EP_8x8mm_P0.4mm_EP6.4x6.4mm, symbol MCU_ST_STM32WB:STM32WB55RGVx
- removed U11: SX1262IMLTRT, lcsc:QFN-24_L4.0-W4.0-P0.50-BL-EP2.6, symbol lcsc:SX1262IMLTRT
- removed U17, U19: NX2012SA-32.768KHZ-STD-MUB-2, lcsc:CRYSTAL-SMD_L2.0-W1.2, symbol lcsc:NX2012SA-32.768KHZ-STD-MUB-2
- removed U2: STM32F405VGTx, Package_QFP:LQFP-100_14x14mm_P0.5mm, symbol MCU_ST_STM32F4:STM32F405VGTx
- removed U21, U5: BMP581, lcsc:LGA-10_L2.0-W2.0-P0.50-TL_BMP581, symbol lcsc:BMP581
- removed U3: BMI270, lcsc:LGA-14_L3.0-W2.5-P0.50-BR, symbol lcsc:BMI270
- removed U4: BMM350_C17225907, lcsc:WLCSP-9_L1.3-W1.3-R3-C3-P0.40-TL, symbol lcsc:BMM350_C17225907
- removed U6: H3LIS331DLTR, lcsc:LGA-16_L3.0-W3.0-P0.50-BL, symbol lcsc:H3LIS331DLTR
- removed U7: ICM-42688-P, lcsc:LGA-14_L3.0-W2.5-P0.50-TL, symbol lcsc:ICM-42688-P
- removed U8: MAX-M10S-00B, lcsc:SMD-18_L10.1-W9.7-P1.10-TL_SKG09F, symbol lcsc:MAX-M10S-00B
- removed U9: W25Q128JVP, Package_SON:WSON-8-1EP_6x5mm_P1.27mm_EP3.4x4.3mm, symbol Memory_Flash:W25Q128JVP
- removed X1: NX2016SA-32MHZ-STD-CZS-5, lcsc:OSC-SMD_4P-L2.0-W1.6-BL, symbol lcsc:NX2016SA-32MHZ-STD-CZS-5
- removed X3: XL2EL89COI-111YLC-24M, lcsc:CRYSTAL-SMD_4P-L3.2-W2.5-BL, symbol lcsc:XL2EL89COI-111YLC-24M
- C28, C29: footprint Capacitor_SMD:C_0603_1608Metric -> Capacitor_SMD:C_0805_2012Metric
Connections:
- net BQ_VREGN is gone; now on net +3.3V: R11.2, R6.2, R7.2
- net GND: now also U18.5 (OTG)
- no-connect marks 26 -> 13
Other:
- added sheet MPU (MPU.kicad_sch)
- added sheet TPU (TPU.kicad_sch)
- moved on the sheet: C19, C20, C21, C22, C23, C24, C25, C26, C27, C28, C29, C31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
