File: hardware/athena.kicad_pcb (KiCad board)
At the start: 2 copper layers, 153 parts, among them SW1 SW_Push, SW2 SW_Push, U1 XL-1608RGBC, U10 STM32WB55RGVx, U11 SX1262IMLTRT, U12 TPS7A2033PDBVR, U13 TPS563209DDCR, U14 XL-1608RGBC, U16 TPD2EUSB30, U17 NX2012SA-32.768KHZ-STD-MUB-2, U18 BQ25886RGE, U19 NX2012SA-32.768KHZ-STD-MUB-2, U2 STM32F405VGTx, U20 USB2422T-I/MJ, U21 BMP581, U22 SZYY0402Y_C434450, U3 BMI270, U4 BMM350_C17225907, U5 BMP581, U6 H3LIS331DLTR, U7 ICM-42688-P, U8 MAX-M10S-00B, U9 W25Q128JVP, X1 NX2016SA-32MHZ-STD-CZS-5, X2 XL2EL89COI-111YLC-24M, X3 XL2EL89COI-111YLC-24M

Commit message: more stuffx
Parts:
- removed C48, C50, C54, C55, C56, C57, C58, C61: 100nF, Capacitor_SMD:C_0402_1005Metric
- removed U21: BMP581, lcsc:LGA-10_L2.0-W2.0-P0.50-TL_BMP581
- added C70: 100nF, Capacitor_SMD:C_0402_1005Metric, F.Cu at (151.5, 88.8)
- added C71: 100nF, Capacitor_SMD:C_0402_1005Metric, F.Cu at (150.0, 89.4)
- added C72: 100nF, Capacitor_SMD:C_0402_1005Metric, F.Cu at (150.8, 107.2)
- added C73: 100nF, Capacitor_SMD:C_0402_1005Metric, F.Cu at (148.8, 107.2)
- added C74: 10nF, Capacitor_SMD:C_0402_1005Metric, F.Cu at (150.3, 112.9)
- added C75: 100nF, Capacitor_SMD:C_0402_1005Metric, F.Cu at (148.0, 113.5)
- added C76: 2.2uF, Capacitor_SMD:C_0402_1005Metric, F.Cu at (146.8, 113.5)
- added C77: 10pF, Capacitor_SMD:C_0402_1005Metric, F.Cu at (127.7, 90.7)
- added C78: 10pF, Capacitor_SMD:C_0402_1005Metric, F.Cu at (127.7, 95.3)
- added C79: 1uF, Capacitor_SMD:C_0402_1005Metric_Pad0.74x0.62mm_HandSolder, F.Cu at (127.8, 88.6)
- added C80: 100nF, Capacitor_SMD:C_0402_1005Metric, F.Cu at (133.2, 94.4)
- added C81: 470nF, Capacitor_SMD:C_0402_1005Metric, F.Cu at (130.4, 94.7)
- added C82: 47nF X7R, Capacitor_SMD:C_0402_1005Metric, F.Cu at (129.2, 88.0)
- added C83: 47pF C0G, Capacitor_SMD:C_0402_1005Metric, F.Cu at (129.2, 87.0)
- added C84: 3pF C0G, Capacitor_SMD:C_0402_1005Metric, F.Cu at (130.7, 84.6)
- added C85: 5.6pF C0G, Capacitor_SMD:C_0402_1005Metric, F.Cu at (130.2, 83.1)
- added C86: 39pF C0G, Capacitor_SMD:C_0402_1005Metric, F.Cu at (130.7, 81.6)
- added C87: 1.8pF C0G, Capacitor_SMD:C_0402_1005Metric, F.Cu at (130.2, 78.4)
- added C88: 1.8pF C0G, Capacitor_SMD:C_0402_1005Metric, F.Cu at (132.7, 86.6)
- added C89: 2.4pF C0G, Capacitor_SMD:C_0402_1005Metric, F.Cu at (131.7, 86.6)
- added C90: 47pF C0G, Capacitor_SMD:C_0402_1005Metric, F.Cu at (129.0, 75.5)
- added C91: 47pF C0G, Capacitor_SMD:C_0402_1005Metric, F.Cu at (134.2, 75.5)
- added C92: 3.3pF C0G, Capacitor_SMD:C_0402_1005Metric, F.Cu at (132.1, 72.1)
- added C93: 39pF C0G, Capacitor_SMD:C_0402_1005Metric, F.Cu at (131.6, 73.7)
- added C94: 3.3pF C0G, Capacitor_SMD:C_0402_1005Metric, F.Cu at (132.1, 69.3)
- added C95: 100nF, Capacitor_SMD:C_0402_1005Metric, F.Cu at (137.0, 79.6)
- added C96: 100nF, Capacitor_SMD:C_0402_1005Metric, F.Cu at (138.6, 79.1)
- added C97: 100nF, Capacitor_SMD:C_0402_1005Metric, F.Cu at (128.6, 102.2)
- added JP1: U.FL-R-SMT-1, lcsc:RF-SMD_FRF05002-JSS103M, F.Cu at (128.5, 119.9)
- added L10: LQW15AN2N5B00D, lcsc:L0402, F.Cu at (129.8, 84.6)
- added L11: LQW15AN4N7C00D, lcsc:L0402, F.Cu at (130.7, 79.8)
- added L12: LQW15AN9N1G00D, lcsc:L0402, F.Cu at (131.6, 70.7)
- added L4: LQW15AN15NG00D, lcsc:IND-SMD_L1.0-W0.5-2, F.Cu at (132.2, 88.0)
- added L8: MLZ2012M150WT000, lcsc:L0805, F.Cu at (130.6, 96.7)
- added L9: LQW15AN47NJ00D, lcsc:L0402, F.Cu at (130.3, 86.0)
- added R38: 100R, Resistor_SMD:R_0402_1005Metric, F.Cu at (129.0, 76.5)
- added R41: 0K, Resistor_SMD:R_0402_1005Metric, F.Cu at (130.7, 87.5)
- added R42: 100R, Resistor_SMD:R_0402_1005Metric, F.Cu at (134.2, 76.5)
- added TP10: TestPoint, custom:TestPoint_Pill, B.Cu at (151.7, 94.4)
- added TP11: TestPoint, custom:TestPoint_Pill, B.Cu at (151.7, 97.8)
- added TP12: TestPoint, custom:TestPoint_Pill, B.Cu at (151.7, 101.3)
- added TP13: TestPoint, custom:TestPoint_Pill, B.Cu at (151.5, 118.5)
- added TP14: TestPoint, custom:TestPoint_Pill, B.Cu at (151.5, 122.0)
- added TP4: TestPoint, TestPoint:TestPoint_Pad_1.0x1.0mm, B.Cu at (52.0, 129.3)
- added TP5: TestPoint, TestPoint:TestPoint_Pad_1.0x1.0mm, B.Cu at (55.1, 129.3)
- added TP6: TestPoint, TestPoint:TestPoint_Pad_1.0x1.0mm, B.Cu at (58.1, 129.3)
- added TP7: TestPoint, custom:TestPoint_Pill, B.Cu at (151.7, 84.0)
- added TP8: TestPoint, custom:TestPoint_Pill, B.Cu at (151.7, 87.5)
- added TP9: TestPoint, custom:TestPoint_Pill, B.Cu at (151.7, 90.9)
- added U15: PE4259-63, lcsc:SC-70-6_L2.2-W1.3-P0.65-LS2.1-BL, F.Cu at (131.6, 76.3)
- added U23: MAX-M10S, RF_GPS:ublox_MAX, F.Cu at (131.8, 108.8)
- added X4: NX2016SA-32MHZ-STD-CZS-5, lcsc:OSC-SMD_4P-L2.0-W1.6-BL, F.Cu at (127.7, 93.0)
- C10, C11, C12, C13, C14, C16, C30, C33, C34, C35, C36, C37, C38, C39, C40, C41, C42, C43, C44, C45, C46, C47, C49, C5, C51, C52, C53, C59, C6, C60, C63, C65, C66, C67, C8, Card1, L6, R17, R18, R19, R20, R21, R22, R29, R30, R31, R32, R33, R34, R39, R40, U19, U2, U20, U4, X2, X3: moved to B.Cu
- C28, C29: footprint Capacitor_SMD:C_0603_1608Metric -> Capacitor_SMD:C_0805_2012Metric
- U11: footprint lcsc:QFN-24_L4.0-W4.0-P0.50-BL-EP2.6 -> Package_DFN_QFN:QFN-24-1EP_4x4mm_P0.5mm_EP2.6x2.6mm
- U8: value MAX-M10S-00B -> BMP581; footprint lcsc:SMD-18_L10.1-W9.7-P1.10-TL_SKG09F -> lcsc:LGA-10_L2.0-W2.0-P0.50-TL_BMP581
- moved FL1 135.8 mm to (232.6, 66.5)
- moved TP1 108.5 mm to (198.3, 68.5)
- moved TP2 108.5 mm to (198.3, 71.6)
- moved TP3 108.5 mm to (198.3, 74.7)
- moved C14 80.5 mm to (149.0, 68.9)
- moved C60 79.5 mm to (129.2, 112.2), turned to -90 degrees
- moved C3 78.9 mm to (144.3, 63.6), turned to 180 degrees
- moved C10 76.2 mm to (146.4, 66.4), turned to 90 degrees
- moved C59 76.1 mm to (131.9, 103.2), turned to 180 degrees
- moved C2 74.8 mm to (142.3, 65.2), turned to 90 degrees
- moved X1 73.9 mm to (144.3, 65.2)
- moved R20 73.6 mm to (129.8, 138.9), turned to -90 degrees
- moved C13 73.4 mm to (149.7, 76.7), turned to -90 degrees
- moved C51 72.5 mm to (129.6, 106.0), turned to 180 degrees
- moved X2 72.0 mm to (131.0, 141.9)
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Connections:
- net /BMI_CS renamed /MPU/BMI_CS
- net /BMI_INT1 renamed /MPU/BMI_INT1
- net /BMI_INT2 renamed /MPU/BMI_INT2
- net /BOOT_MPU renamed BOOT_MPU
- net /BOOT_TPU renamed BOOT_TPU
- net /FLASH_CLK renamed /MPU/FLASH_CLK
- net /FLASH_CS renamed /MPU/FLASH_CS
- net /FLASH_MISO renamed /MPU/FLASH_MISO
- net /FLASH_MOSI renamed /MPU/FLASH_MOSI
- net /FLASH_SCK renamed /MPU/FLASH_SCK
- net /MAG_INT renamed /MPU/MAG_INT
- net /MAG_SCL renamed /MPU/MAG_SCL
- net /MAG_SDA renamed /MPU/MAG_SDA
- net /MPU_B renamed MPU_B
- net /MPU_DN renamed MPU_DN
- net /MPU_DP renamed MPU_DP
- net /MPU_G renamed MPU_G
- net /MPU_HXIN renamed /MPU/MPU_HXIN
- net /MPU_HXOUT renamed /MPU/MPU_HXOUT
- net /MPU_LXIN renamed /MPU/MPU_LXIN
- net /MPU_LXOUT renamed /MPU/MPU_LXOUT
- net /MPU_R renamed MPU_R
- net /RESET_MPU renamed RESET_MPU
- net /RESET_TPU renamed RESET_TPU
- net /RF renamed /TPU/RF
- net /SD_CD renamed /MPU/SD_CD
- net /SD_CLK renamed /MPU/SD_CLK
- net /SD_CMD renamed /MPU/SD_CMD
- net /SD_D0 renamed /MPU/SD_D0
- net /TPU_DN renamed TPU_DN
- net /TPU_DP renamed TPU_DP
- net /TPU_HXIN renamed /TPU/TPU_HXIN
- net /TPU_HXOUT renamed /TPU/TPU_HXOUT
- net /TPU_LXIN renamed /TPU/TPU_LXIN
- net /TPU_LXOUT renamed /TPU/TPU_LXOUT
- net /TPU_SWCLK renamed /TPU/TPU_SWCLK
- net /TPU_SWDIO renamed /TPU/TPU_SWDIO
- R11 pad 2: BQ_VREGN -> +3.3V
- R26 pad 1: /TPU_R -> TPU_R
- R27 pad 2: /TPU_G -> TPU_G
- R28 pad 2: /TPU_B -> TPU_B
- R6 pad 2: BQ_VREGN -> +3.3V
- R7 pad 2: BQ_VREGN -> +3.3V
- RF1 pad 1: unconnected-(RF1-Pad1) -> GND
- RF1 pad 2: unconnected-(RF1-Pad2) -> GND
- RF1 pad 3: unconnected-(RF1-Pad3) -> GND
- RF1 pad 4: unconnected-(RF1-Pad4) -> GND
- RF1 pad 5: unconnected-(RF1-Pad5) -> Net-(C94-Pad1)
- U10 pad 15: unconnected-(U10-PA0-Pad15) -> TPU_R
- U10 pad 16: unconnected-(U10-PA1-Pad16) -> TPU_G
- U10 pad 17: unconnected-(U10-PA2-Pad17) -> TPU_B
- U10 pad 46: unconnected-(U10-PB12-Pad46) -> /TPU/BARO_CS
- U10 pad 47: unconnected-(U10-PB13-Pad47) -> /TPU/BARO_SCK
- U10 pad 48: unconnected-(U10-PB14-Pad48) -> /TPU/BARO_MISO
- U10 pad 49: unconnected-(U10-PB15-Pad49) -> /TPU/BARO_MOSI
- U10 pad 50: unconnected-(U10-PC6-Pad50) -> /TPU/BARO_INT
- U10 pad 66: unconnected-(U10-PB6-Pad66) -> /MPU/MPU_RX
- U10 pad 67: unconnected-(U10-PB7-Pad67) -> /MPU/MPU_TX
- U11 pad 1: unconnected-(U11-VDD_IN-Pad1) -> +3.3V
- U11 pad 10: unconnected-(U11-VBAT-Pad10) -> +3.3V
- U11 pad 11: unconnected-(U11-VBAT_IO-Pad11) -> +3.3V
- U11 pad 12: unconnected-(U11-DIO2-Pad12) -> /TPU/LORA_DIO2
- U11 pad 13: unconnected-(U11-DIO1-Pad13) -> /TPU/LORA_DIO1
- U11 pad 14: unconnected-(U11-BUSY-Pad14) -> /TPU/LORA_BUSY
- U11 pad 15: unconnected-(U11-NRESET-Pad15) -> /TPU/LORA_RESET
- U11 pad 16: unconnected-(U11-MISO-Pad16) -> /TPU/LORA_MISO
- U11 pad 17: unconnected-(U11-MOSI-Pad17) -> /TPU/LORA_MOSI
- U11 pad 18: unconnected-(U11-SCK-Pad18) -> /TPU/LORA_SCK
- U11 pad 19: unconnected-(U11-NSS-Pad19) -> /TPU/LORA_CS
- U11 pad 2: unconnected-(U11-GND-Pad2) -> GND
- U11 pad 20: unconnected-(U11-GND-Pad20) -> GND
- U11 pad 21: unconnected-(U11-RFI_P-Pad21) -> Net-(U11-RFI_P)
- U11 pad 22: unconnected-(U11-RFI_N-Pad22) -> Net-(U11-RFI_N)
- U11 pad 23: unconnected-(U11-RFO-Pad23) -> Net-(U11-RFO)
- U11 pad 24: unconnected-(U11-VR_PA-Pad24) -> Net-(U11-VR_PA)
- U11 pad 25: unconnected-(U11-GND-Pad25) -> GND
- U11 pad 3: unconnected-(U11-XTA-Pad3) -> /TPU/LORA_XIN
- U11 pad 4: unconnected-(U11-XTB-Pad4) -> /TPU/LORA_XOUT
- U11 pad 5: unconnected-(U11-GND-Pad5) -> GND
- U11 pad 6: unconnected-(U11-DIO3-Pad6) -> /TPU/LORA_DIO3
- U11 pad 7: unconnected-(U11-VREG-Pad7) -> Net-(U11-VREG)
- U11 pad 8: unconnected-(U11-GND-Pad8) -> GND
- U11 pad 9: unconnected-(U11-DCC_SW-Pad9) -> Net-(U11-DCC_SW)
- U18 pad 5: unconnected-(U18-OTG-Pad5) -> GND
- U2 pad 30: /IMU_SCK -> /MPU/IMU_SCK
- U2 pad 31: /IMU_MISO -> /MPU/IMU_MISO
- U2 pad 32: /IMU_MOSI -> /MPU/IMU_MOSI
- U2 pad 37: unconnected-(U2-PB2-Pad37) -> /MPU/ICM_CS
- U2 pad 38: unconnected-(U2-PE7-Pad38) -> /MPU/ICM_INT1
- U2 pad 39: unconnected-(U2-PE8-Pad39) -> /MPU/ICM_INT2
- U2 pad 40: /MOTOR_1 -> /MPU/MOTOR_1
- U2 pad 42: /MOTOR_2 -> /MPU/MOTOR_2
- U2 pad 44: /MOTOR_3 -> /MPU/MOTOR_3
- U2 pad 45: /MOTOR_4 -> /MPU/MOTOR_4
- U2 pad 52: /SENSOR_SCK -> /MPU/SENSOR_SCK
- U2 pad 53: /SENSOR_MISO -> /MPU/SENSOR_MISO
- U2 pad 54: /SENSOR_MOSI -> /MPU/SENSOR_MOSI
- U2 pad 55: unconnected-(U2-PD8-Pad55) -> /MPU/BMP_CS
- U2 pad 56: unconnected-(U2-PD9-Pad56) -> /MPU/BMP_INT
- U2 pad 57: unconnected-(U2-PD10-Pad57) -> /MPU/HLI_CS
- U2 pad 58: unconnected-(U2-PD11-Pad58) -> /MPU/HLI_INT1
- U2 pad 59: unconnected-(U2-PD12-Pad59) -> /MPU/HLI_INT2
- U2 pad 63: /MOTOR_5 -> /MPU/MOTOR_5
- U2 pad 64: /MOTOR_6 -> /MPU/MOTOR_6
- U2 pad 66: /MOTOR_8 -> /MPU/MOTOR_8
- U2 pad 68: /TPU_TX -> /MPU/MPU_TX
- U2 pad 69: /TPU_RX -> /MPU/MPU_RX
- U2 pad 72: /MPU_SWDIO -> /MPU/MPU_SWDIO
- U2 pad 76: /MPU_SWCLK -> /MPU/MPU_SWCLK
- U2 pad 84: unconnected-(U2-PD3-Pad84) -> /MPU/GPS_EXTINT
- U2 pad 85: unconnected-(U2-PD4-Pad85) -> /MPU/GPS_SAFEBOOT
- U2 pad 86: /GPS_TX -> /MPU/GPS_TX
- U2 pad 87: /GPS_RX -> /MPU/GPS_RX
- U2 pad 88: unconnected-(U2-PD7-Pad88) -> /MPU/GPS_RESET
- U2 pad 93: /MOTOR_7 -> /MPU/MOTOR_7
- U3 pad 1: /IMU_MISO -> /MPU/IMU_MISO
- U3 pad 13: /IMU_SCK -> /MPU/IMU_SCK
- U3 pad 14: /IMU_MOSI -> /MPU/IMU_MOSI
- U5 pad 1: unconnected-(U5-VDDIO-Pad1) -> +3.3V_LDO
- U5 pad 10: unconnected-(U5-VDD-Pad10) -> +3.3V_LDO
- U5 pad 2: unconnected-(U5-SCK-Pad2) -> /MPU/SENSOR_SCK
- U5 pad 3: unconnected-(U5-VSS-Pad3) -> GND
- U5 pad 4: unconnected-(U5-SDI-Pad4) -> /MPU/SENSOR_MOSI
- U5 pad 5: unconnected-(U5-SDO-Pad5) -> /MPU/SENSOR_MISO
- U5 pad 6: unconnected-(U5-CSB-Pad6) -> /MPU/BMP_CS
- U5 pad 7: unconnected-(U5-INT-Pad7) -> /MPU/BMP_INT
- U5 pad 8: unconnected-(U5-VSS-Pad8) -> GND
- U5 pad 9: unconnected-(U5-VSS-Pad9) -> GND
- U6 pad 1: unconnected-(U6-Vdd_IO-Pad1) -> +3.3V_LDO
- U6 pad 10: unconnected-(U6-Reserved-Pad10) -> GND
- U6 pad 11: unconnected-(U6-INT1-Pad11) -> /MPU/HLI_INT1
- U6 pad 12: unconnected-(U6-GND-Pad12) -> GND
- U6 pad 13: unconnected-(U6-GND-Pad13) -> GND
- U6 pad 14: unconnected-(U6-Vdd-Pad14) -> +3.3V_LDO
- U6 pad 15: unconnected-(U6-Reserved-Pad15) -> GND
- U6 pad 16: unconnected-(U6-GND-Pad16) -> GND
- U6 pad 4: unconnected-(U6-SCL/SPS-Pad4) -> /MPU/SENSOR_SCK
- U6 pad 5: unconnected-(U6-GND-Pad5) -> GND
- U6 pad 6: unconnected-(U6-SDA/SDI/SDO-Pad6) -> /MPU/SENSOR_MOSI
- U6 pad 7: unconnected-(U6-SDO/SA0-Pad7) -> /MPU/SENSOR_MISO
- U6 pad 8: unconnected-(U6-CS-Pad8) -> /MPU/HLI_CS
- U6 pad 9: unconnected-(U6-INT2-Pad9) -> /MPU/HLI_INT2
- U7 pad 1: unconnected-(U7-AP_SDO/AP_AD0-Pad1) -> /MPU/IMU_MISO
- U7 pad 12: unconnected-(U7-AP_CS-Pad12) -> /MPU/ICM_CS
- U7 pad 13: unconnected-(U7-AP_SCL/AP_SCLK-Pad13) -> /MPU/IMU_SCK
- U7 pad 14: unconnected-(U7-AP_SDA/AP_SDIO/AP_SDI-Pad14) -> /MPU/IMU_MOSI
- U7 pad 4: unconnected-(U7-INT1/INT-Pad4) -> /MPU/ICM_INT1
- U7 pad 5: unconnected-(U7-VDDIO-Pad5) -> +3.3V_LDO
- U7 pad 6: unconnected-(U7-GND-Pad6) -> GND
- U7 pad 8: unconnected-(U7-VDD-Pad8) -> +3.3V_LDO
- U7 pad 9: unconnected-(U7-INT2/FSYNC/CLKIN-Pad9) -> /MPU/ICM_INT2
- U8 pad 1: unconnected-(U8-GND-Pad1) -> +3.3V
- U8 pad 10: unconnected-(U8-GND-Pad10) -> +3.3V
- U8 pad 2: unconnected-(U8-TXD-Pad2) -> /TPU/BARO_SCK
- U8 pad 3: unconnected-(U8-RXD-Pad3) -> GND
- U8 pad 4: unconnected-(U8-TIMEPULSE-Pad4) -> /TPU/BARO_MOSI
- U8 pad 5: unconnected-(U8-EXTINT-Pad5) -> /TPU/BARO_MISO
- U8 pad 6: unconnected-(U8-V_BCKP-Pad6) -> /TPU/BARO_CS
- U8 pad 7: unconnected-(U8-V_IO-Pad7) -> /TPU/BARO_INT
- U8 pad 8: unconnected-(U8-VCC-Pad8) -> GND
- U8 pad 9: unconnected-(U8-RESET_N-Pad9) -> GND
Other:
- board outline added: 30 x 90 mm
- copper layers 2 -> 4
- board text added: "Athena V2"
